File: pcb/trone.kicad_pcb (KiCad board)
At the start: 2 copper layers, 135.2 x 89 mm, 42 parts

Commit message: fully routed
Parts:
- removed REF**: USB_C_Receptacle_Amphenol_12401548E4-2A, Connector_USB:USB_C_Receptacle_Amphenol_12401548E4-2A
- added J1: Jumper, lib:Jumper, F.Cu at (0.00, 0.00)
- added USBC1: , AMPHENOL_12401548E4#2A, F.Cu at (266.9, 150.9)
Routing:
- net P15: track 20.3 -> 246.8 mm
- net P18: track 20.3 -> 219.7 mm
- net P19: track 150.0 -> 342.9 mm
- net P14: track 20.6 -> 192.9 mm
- net P16: track 43.4 -> 167.0 mm
- net P7: track 0.00 -> 50.0 mm
- net P0: track 152.0 -> 189.0 mm
- net P10: track 102.5 -> 138.1 mm
- net P6: track 0.00 -> 35.2 mm
- net P4: track 159.1 -> 188.8 mm
- net P1: track 238.9 -> 265.5 mm
- net P9: track 0.00 -> 23.2 mm
- net P5: track 0.00 -> 21.8 mm
- net GND: track 0.00 -> 18.8 mm
- net P8: track 0.00 -> 14.9 mm
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Other:
- outline, holes or cut-outs redrawn
