File: pcbs/trone.kicad_pcb (KiCad board)
At the start: 2 copper layers, 135.2 x 87 mm, 56 parts, among them J1 Jumper

Commit message: done
Parts:
- removed J1: Jumper, lib:Jumper
- removed the REF** at (182.3, 160.5)
Connections:
- SW1 pad 1: RAW -> VCC
- SW1 pad 2: P1 -> RAW
Routing:
- net P1: track 163.1 -> 0.00 mm
- net RAW: track 290.7 -> 204.0 mm
- net COL4: track 242.7 -> 272.2 mm
- net VCC: track 234.3 -> 257.1 mm
- net COL3: track 346.6 -> 366.4 mm
- net RST: track 7.07 -> 0.00 mm
- net GND: track 557.2 -> 563.3 mm
- net COL1: track 202.7 -> 203.7 mm
Other:
- outline, holes or cut-outs redrawn
